File: hardware/kicad/LED_Module_CH32V203.kicad_sch (KiCad schematic)
At the start: 96 parts, among them J1 USB_C_Receptacle_USB2.0_16P, J2 Solder Pad, J3 Qwiic / StemmaQT Connector, J4 noknok_FlashPads_USB-module, Q1 AO3401A, Q2 MMBT3904, U1 CH32V203G6U6, U2 BL9110-330BPFB (LCSC C169246), U3 SN74AHCT1G125DBVR (LCSC C7484), Y1 Crystal

Commit message: hardware: revert to the 8x WS2812b board - the 16x SK6812 rev2 design moves to module-usb-led-16x
Parts:
- removed C19, C24: 10uF, Capacitor_SMD:C_0603_1608Metric, symbol Device:C
- removed C20, C21, C22, C23, C27, C28, C33, C34, C35, C38: 0.1uF, Capacitor_SMD:C_0603_1608Metric, symbol Device:C
- removed C29, C32, C36, C37: 22µF 25V X5R, Capacitor_SMD:C_1206_3216Metric, symbol Device:C
- removed C30, C39, C40, C41: 0.1uF X7R Ceramic, Capacitor_SMD:C_0603_1608Metric, symbol Device:C
- removed C31: 0.1uF X7R 16V+, Capacitor_SMD:C_0603_1608Metric, symbol Device:C
- removed D1: PMEG4010CEH (LCSC C193342), Diode_SMD:D_SOD-123, symbol Device:D_Schottky
- removed D17, D18, D19, D20, D21, D22, D23, D24: SK6812, LED_SMD:LED_SK6812_PLCC4_5.0x5.0mm_P3.2mm, symbol LED:SK6812
- removed D5: LED, LED_SMD:LED_0603_1608Metric, symbol Device:LED
- removed H1, H2, H3: noknok_MountingHole, noknok:noknok_MountingHole_2.5mm_M2.5, symbol noknok:noknok_MountingHole
- removed J4: noknok_FlashPads_USB-module, noknok:noknok_FlashPads_USB-module_1x4_M2.5, symbol noknok:noknok_FlashPads_USB-module
- removed Q1: AO3401A, Package_TO_SOT_SMD:SOT-23, symbol Transistor_FET:AO3401A
- removed Q2: MMBT3904, Package_TO_SOT_SMD:SOT-23, symbol Transistor_BJT:MMBT3904
- removed R10: 2.2k, Resistor_SMD:R_0603_1608Metric, symbol Device:R
- removed R11, R12, R13, R14: 10k, Resistor_SMD:R_0603_1608Metric, symbol Device:R
- removed R15: 1k, Resistor_SMD:R_0603_1608Metric, symbol Device:R
- removed R16, R17: 22k, Resistor_SMD:R_0603_1608Metric, symbol Device:R
- removed R18, R19: 4.7k (1% tolerance), Resistor_SMD:R_0603_1608Metric, symbol Device:R
- removed R20, R21: 3.3k (1% tolerance), Resistor_SMD:R_0603_1608Metric, symbol Device:R
- removed U2: BL9110-330BPFB (LCSC C169246), Package_TO_SOT_SMD:SOT-223-3_TabPin2, symbol Regulator_Linear:AMS1117-3.3
- removed U3: SN74AHCT1G125DBVR (LCSC C7484), Package_TO_SOT_SMD:SOT-23-5, symbol 74xGxx:74AHC1G125
- added D1: 1N4007, Diode_SMD:D_SOD-123, symbol Diode:1N4007
- added J4: Qwiic / StemmaQT Connector, Connector_JST:JST_SH_BM04B-SRSS-TB_1x04-1MP_P1.00mm_Vertical, symbol Connector_Generic:Conn_01x04
- added J5: TagConnect_TC2030, Connector:Tag-Connect_TC2030-IDC-NL_2x03_P1.27mm_Vertical, symbol Connector:Conn_ARM_SWD_TagConnect_TC2030-NL
- added TP1: TestPoint, TestPoint:TestPoint_THTPad_D1.0mm_Drill0.5mm, symbol Connector:TestPoint
- added U2: XC6206P332MR, Package_TO_SOT_SMD:SOT-23-3, symbol Regulator_Linear:XC6206PxxxMR
- C1, C10, C11, C12, C13, C14, C15, C16, C17, C18, C2, C3, C4, C5, C6, C7, C8, C9: footprint Capacitor_SMD:C_0603_1608Metric -> Capacitor_SMD:C_0603_1608Metric_Pad1.08x0.95mm_HandSolder
- D10, D11, D12, D13, D14, D15, D16, D9: value SK6812 -> WS2812B; footprint LED_SMD:LED_SK6812_PLCC4_5.0x5.0mm_P3.2mm -> LED_SMD:LED_WS2812B_PLCC4_5.0x5.0mm_P3.2mm; symbol LED:SK6812 -> LED:WS2812B
- D4: footprint Diode_SMD:D_SOD-323 -> Diode_SMD:D_SOD-323_HandSoldering
- F1: value Polyfuse at >= 2A -> Resettable Polyfuse
- J1: footprint (none) -> Connector_USB:USB_C_Receptacle_GCT_USB4105-xx-A_16P_TopMnt_Horizontal
- J2: value Solder Pad -> Jumper Cap; footprint Jumper:SolderJumper-2_P1.3mm_Open_TrianglePad1.0x1.5mm -> Connector_PinHeader_2.54mm:PinHeader_1x02_P2.54mm_Vertical
- R1, R2: value 1.8k (1% tolerance) -> 5.1k; footprint Resistor_SMD:R_0603_1608Metric -> Resistor_SMD:R_0603_1608Metric_Pad0.98x0.95mm_HandSolder
- R3, R4, R5, R6, R7: footprint Resistor_SMD:R_0603_1608Metric -> Resistor_SMD:R_0603_1608Metric_Pad0.98x0.95mm_HandSolder
- R8, R9: value 3.3k -> 4.7k; footprint Resistor_SMD:R_0603_1608Metric -> Resistor_SMD:R_0603_1608Metric_Pad0.98x0.95mm_HandSolder
- Y1: footprint Crystal:Crystal_SMD_3225-4Pin_3.2x2.5mm -> Crystal:Crystal_SMD_3225-4Pin_3.2x2.5mm_HandSoldering
Connections:
- net D_N is gone; now on net D-: R3.1, U1.19 (PA10/PA11/USB_D-)
- net D_P is gone; now on net D+: R4.1, U1.20 (PA12/USB_D+)
- net MCU_PA3 is gone; now on an unnamed net: U1.9 (PA3)
- net +3.3V: now also J4.2 (Pin_2), J5.1 (VCC), U2.2 (VO)
- net +5V: now also D1.2 (A)
- net GND: now also D10.3 (VSS), D11.3 (VSS), D12.3 (VSS), D13.3 (VSS), D14.3 (VSS), D15.3 (VSS), D16.3 (VSS), D9.3 (VSS), J1.S1 (SHIELD), J4.1 (Pin_1), J5.5 (GND), U2.1 (GND); no longer D10.1 (VSS), D11.1 (VSS), D12.1 (VSS), D13.1 (VSS), D14.1 (VSS), D15.1 (VSS), D16.1 (VSS), D9.1 (VSS), J1.SH (SHIELD)
- net at U1.21 (PA13/SWDIO): now also J5.2 (SWDIO)
- net at U1.22 (PA14/SWCLK): now also J5.4 (SWCLK)
- net at J3.4 (Pin_4), R8.1, U1.27 (PB6): now also J4.4 (Pin_4)
- net at J3.3 (Pin_3), R9.1, U1.28 (PB7): now also J4.3 (Pin_3)
- net at C6.2, R6.1, U1.4 (~{RST}): now also J5.3 (~{RESET})
- net at D10.2 (DOUT): now also D11.4 (DIN); no longer D9.4 (DOUT)
- net at D10.4 (DIN): now also D9.2 (DOUT); no longer D11.2 (DIN)
- net at D12.2 (DOUT): now also D13.4 (DIN); no longer D11.4 (DOUT)
- net at D16.4 (DIN): now also D15.2 (DOUT)
- net at R2.2: now also J1.B5 (CC2)
- net at D12.4 (DIN): now also D11.2 (DOUT); no longer D13.2 (DIN)
- net at D14.2 (DOUT): now also D15.4 (DIN); no longer D13.4 (DOUT)
- net at D14.4 (DIN): now also D13.2 (DOUT); no longer D15.2 (DIN)
- net at R1.2: now also J1.A5 (CC1)
- net at D16.2 (DOUT): no longer D15.4 (DOUT)
- net +4.65V renamed +4.1V
- net +4.1V: now also C1.1, C10.1, C11.1, C12.1, C13.1, C14.1, C15.1, C16.1, C8.1, C9.1, D10.1 (VDD), D11.1 (VDD), D12.1 (VDD), D13.1 (VDD), D14.1 (VDD), D15.1 (VDD), D16.1 (VDD), D9.1 (VDD), D1.1 (K), TP1.1, U2.3 (VI)
- removed net +5V_LED: C1.1, C10.1, C11.1, C12.1, C13.1, C14.1, C15.1, C16.1, C8.1, C9.1, D10.3 (VDD), D11.3 (VDD), D12.3 (VDD), D13.3 (VDD), D14.3 (VDD), D15.3 (VDD), D16.3 (VDD), D9.3 (VDD)
- net D9_DIN: no longer names the net of R5.1, TP2.1
- net D9_DIN: now also D9.4 (DIN); no longer D9.2 (DIN)
- net MCU_PA0: no longer names the net of U1.6 (PA0)
- net MCU_PA1: no longer names the net of U1.7 (PA1)
- net MCU_PA2: no longer names the net of U1.8 (PA2)
- net MCU_PB0: no longer names the net of U1.14 (PB0)
- no-connect marks 13 -> 18
Other:
- note added: ""big" power reservoir for 4 WS2812b to stabilize"
- note added: "Bulk capacitors for XC6206P"
- note added: "Convert 4.1V to 3.3V"
- note added: "Decoupling capacitor for MCU"
- note added: "bypass capacitor for each WS2812B to stabilize power"
- note added: "decoupling capacitor for 4 WS2812b to stabilize"
- note added: "protect XC6206P reverse charge"
- note removed: ""big" power reservoir for 4 SK6812 to stabilize"
- note removed: "AO3401 is a power on/off switch. MMBT3904 allows MCU to switch on power for SK6812 by driving PB0 high or low (helps brownout protection at power on)"
- note removed: "Convert 4.65V to 3.3V for MCU"
- note removed: "Decoupling capacitors for MCU"
- note removed: "Measure CC voltage"
- note removed: "Status Indicator LED (active high)"
- note removed: "USB LEDs Module 16x SK6812 RGBW"
- note removed: "VBUS sensing, measure voltage (could be left unpopulated)"
- note removed: "WS2812 decides "1" at 0.7 of own supply voltage. Supply voltage at 5V, *0.7 = 3.5V threshold. MCU sends a "1" at 3.3V -> below threshold, LED would never see a "1". This chip "converts" data signal from MCU to a clear +5V for "1" so data signal is unambiguous towards SK6812."
- note removed: "bypass capacitor for each SK6812 to stabilize power"
- note removed: "optional to add Ferrite Bead (600R@100Mhz - LCSC C275451) between 3.3V and VDDA to improve ADC for USB sensing"
- note removed: "protect BL9110 reverse charge"
- title: USB-C LEDs Module -> USB-C LED Module
- moved on the sheet: C1, C10, C11, C12, C13, C14, C15, C16, C17, C18, C2, C3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

Commit message: hardware: rev 2.0 round board with 16x SKC6812RGBW, add BOM and schematic PDF, drop stale renders
Parts:
- removed D1: 1N4007, Diode_SMD:D_SOD-123, symbol Diode:1N4007
- removed J4: Qwiic / StemmaQT Connector, Connector_JST:JST_SH_BM04B-SRSS-TB_1x04-1MP_P1.00mm_Vertical, symbol Connector_Generic:Conn_01x04
- removed J5: TagConnect_TC2030, Connector:Tag-Connect_TC2030-IDC-NL_2x03_P1.27mm_Vertical, symbol Connector:Conn_ARM_SWD_TagConnect_TC2030-NL
- removed TP1: TestPoint, TestPoint:TestPoint_THTPad_D1.0mm_Drill0.5mm, symbol Connector:TestPoint
- removed U2: XC6206P332MR, Package_TO_SOT_SMD:SOT-23-3, symbol Regulator_Linear:XC6206PxxxMR
- added C19, C24: 10uF, Capacitor_SMD:C_0603_1608Metric, symbol Device:C
- added C20, C21, C22, C23, C27, C28, C33, C34, C35, C38: 0.1uF, Capacitor_SMD:C_0603_1608Metric, symbol Device:C
- added C29, C32, C36, C37: 22µF 25V X5R, Capacitor_SMD:C_1206_3216Metric, symbol Device:C
- added C30, C39, C40, C41: 0.1uF X7R Ceramic, Capacitor_SMD:C_0603_1608Metric, symbol Device:C
- added C31: 0.1uF X7R 16V+, Capacitor_SMD:C_0603_1608Metric, symbol Device:C
- added D1: PMEG4010CEH (LCSC C193342), Diode_SMD:D_SOD-123, symbol Device:D_Schottky
- added D17, D18, D19, D20, D21, D22, D23, D24: SK6812, LED_SMD:LED_SK6812_PLCC4_5.0x5.0mm_P3.2mm, symbol LED:SK6812
- added D5: LED, LED_SMD:LED_0603_1608Metric, symbol Device:LED
- added H1, H2, H3: noknok_MountingHole, noknok:noknok_MountingHole_2.5mm_M2.5, symbol noknok:noknok_MountingHole
- added J4: noknok_FlashPads_USB-module, noknok:noknok_FlashPads_USB-module_1x4_M2.5, symbol noknok:noknok_FlashPads_USB-module
- added Q1: AO3401A, Package_TO_SOT_SMD:SOT-23, symbol Transistor_FET:AO3401A
- added Q2: MMBT3904, Package_TO_SOT_SMD:SOT-23, symbol Transistor_BJT:MMBT3904
- added R10: 2.2k, Resistor_SMD:R_0603_1608Metric, symbol Device:R
- added R11, R12, R13, R14: 10k, Resistor_SMD:R_0603_1608Metric, symbol Device:R
- added R15: 1k, Resistor_SMD:R_0603_1608Metric, symbol Device:R
- added R16, R17: 22k, Resistor_SMD:R_0603_1608Metric, symbol Device:R
- added R18, R19: 4.7k (1% tolerance), Resistor_SMD:R_0603_1608Metric, symbol Device:R
- added R20, R21: 3.3k (1% tolerance), Resistor_SMD:R_0603_1608Metric, symbol Device:R
- added U2: BL9110-330BPFB (LCSC C169246), Package_TO_SOT_SMD:SOT-223-3_TabPin2, symbol Regulator_Linear:AMS1117-3.3
- added U3: SN74AHCT1G125DBVR (LCSC C7484), Package_TO_SOT_SMD:SOT-23-5, symbol 74xGxx:74AHC1G125
- C1, C10, C11, C12, C13, C14, C15, C16, C17, C18, C2, C3, C4, C5, C6, C7, C8, C9: footprint Capacitor_SMD:C_0603_1608Metric_Pad1.08x0.95mm_HandSolder -> Capacitor_SMD:C_0603_1608Metric
- D10, D11, D12, D13, D14, D15, D16, D9: value WS2812B -> SK6812; footprint LED_SMD:LED_WS2812B_PLCC4_5.0x5.0mm_P3.2mm -> LED_SMD:LED_SK6812_PLCC4_5.0x5.0mm_P3.2mm; symbol LED:WS2812B -> LED:SK6812
- D4: footprint Diode_SMD:D_SOD-323_HandSoldering -> Diode_SMD:D_SOD-323
- F1: value Resettable Polyfuse -> Polyfuse at >= 2A
- J1: footprint Connector_USB:USB_C_Receptacle_GCT_USB4105-xx-A_16P_TopMnt_Horizontal -> (none)
- J2: value Jumper Cap -> Solder Pad; footprint Connector_PinHeader_2.54mm:PinHeader_1x02_P2.54mm_Vertical -> Jumper:SolderJumper-2_P1.3mm_Open_TrianglePad1.0x1.5mm
- R1, R2: value 5.1k -> 1.8k (1% tolerance); footprint Resistor_SMD:R_0603_1608Metric_Pad0.98x0.95mm_HandSolder -> Resistor_SMD:R_0603_1608Metric
- R3, R4, R5, R6, R7: footprint Resistor_SMD:R_0603_1608Metric_Pad0.98x0.95mm_HandSolder -> Resistor_SMD:R_0603_1608Metric
- R8, R9: value 4.7k -> 3.3k; footprint Resistor_SMD:R_0603_1608Metric_Pad0.98x0.95mm_HandSolder -> Resistor_SMD:R_0603_1608Metric
- Y1: footprint Crystal:Crystal_SMD_3225-4Pin_3.2x2.5mm_HandSoldering -> Crystal:Crystal_SMD_3225-4Pin_3.2x2.5mm
Connections:
- net +3.3V: now also C33.1, C34.2, J4.3 (VCC), U2.2 (VO)
- net +5V: now also C29.1, C30.1, C31.1, C32.1, C36.2, C37.2, D1.2 (A), Q1.2 (S), R11.2, R16.2, U3.5 (VCC)
- net D+: no longer R4.1, U1.20 (PA12/USB_D+)
- net D-: no longer R3.1, U1.19 (PA10/PA11/USB_D-)
- net GND: now also D10.1 (VSS), D11.1 (VSS), D12.1 (VSS), D13.1 (VSS), D14.1 (VSS), D15.1 (VSS), D16.1 (VSS), D9.1 (VSS), J1.SH (SHIELD), C19.2, C20.2, C21.2, C22.2, C23.2, C24.2, C27.2, C28.2, C29.2, C30.2, C31.2, C32.2, C33.2, C34.1, C35.2, C36.1, C37.1, C39.2, C40.2, C41.1, D17.1 (VSS), D18.1 (VSS), D19.1 (VSS), D20.1 (VSS), D21.1 (VSS), D22.1 (VSS), D23.1 (VSS), D24.1 (VSS), D5.1 (K), J4.1 (GND), Q2.2 (E), R12.1, R14.1, R17.2, U2.1 (GND), U3.1, U3.3 (GND); no longer D10.3 (VSS), D11.3 (VSS), D12.3 (VSS), D13.3 (VSS), D14.3 (VSS), D15.3 (VSS), D16.3 (VSS), D9.3 (VSS), J1.S1 (SHIELD)
- net at U1.21 (PA13/SWDIO): now also J4.2 (SWDIO)
- net at U1.22 (PA14/SWCLK): now also J4.4 (SWCLK)
- net at J2.2 (Pin_2), R7.1, U1.1 (BOOT0/PB8): now also R10.2
- net MCU_PB0: now reaches U1.14 (PB0)
- net MCU_PB0: now also R13.1
- net MCU_PA0: now reaches U1.6 (PA0)
- net MCU_PA0: now also C35.1, C41.2, R16.1, R17.1
- net MCU_PA1: now reaches U1.7 (PA1)
- net MCU_PA1: now also C40.1, R18.1
- net MCU_PA2: now reaches U1.8 (PA2)
- net MCU_PA2: now also C39.1, R19.1
- net at R5.2: now also U3.4; no longer U1.9 (PA3)
- net at D10.2 (DIN): now also D9.4 (DOUT); no longer D11.4 (DIN)
- net at D10.4 (DOUT): now also D11.2 (DIN); no longer D9.2 (DOUT)
- net at D12.4 (DOUT): now also D13.2 (DIN); no longer D11.2 (DOUT)
- net D9_DIN: now reaches R5.1, TP2.1
- net D9_DIN: now also D9.2 (DIN); no longer D9.4 (DIN)
- net at D12.2 (DIN): now also D11.4 (DOUT); no longer D13.4 (DIN)
- net at D14.2 (DIN): now also D13.4 (DOUT); no longer D15.4 (DIN)
- net at D14.4 (DOUT): now also D15.2 (DIN); no longer D13.2 (DOUT)
- net at D16.2 (DIN): now also D15.4 (DOUT)
- net at D16.4 (DOUT): now also D17.2 (DIN); no longer D15.2 (DOUT)
- net at R1.2: now also R18.2, R20.1; no longer J1.A5 (CC1)
- net at R2.2: now also R19.2, R21.1; no longer J1.B5 (CC2)
- removed net +4.1V: C1.1, C10.1, C11.1, C12.1, C13.1, C14.1, C15.1, C16.1, C2.1, C3.1, C8.1, C9.1, D10.1 (VDD), D11.1 (VDD), D12.1 (VDD), D13.1 (VDD), D14.1 (VDD), D15.1 (VDD), D16.1 (VDD), D4.1 (K), D9.1 (VDD)
- new net: D17.4 (DOUT), D18.2 (DIN)
- new net: D18.4 (DOUT), D19.2 (DIN)
- new net: D22.4 (DOUT), D23.2 (DIN)
- new net: D23.4 (DOUT), D24.2 (DIN)
- new net: D5.2 (A), R10.1
- new net: C38.2, Q1.1 (G), R11.1, R15.2
- new net: Q2.1 (B), R12.2, R13.2
- new net: Q2.3 (C), R15.1
- new net: D19.4 (DOUT), D20.2 (DIN)
- new net: D20.4 (DOUT), D21.2 (DIN)
- new net: D21.4 (DOUT), D22.2 (DIN)
- new net: J1.A5 (CC1), R20.2
- new net: J1.B5 (CC2), R21.2
- new net +4.65V: C2.1, C3.1, D1.1 (K), D4.1 (K), U2.3 (VI)
- new net +5V_LED: C1.1, C10.1, C11.1, C12.1, C13.1, C14.1, C15.1, C16.1, C19.1, C20.1, C21.1, C22.1, C23.1, C24.1, C27.1, C28.1, C38.1, C8.1, C9.1, D10.3 (VDD), D11.3 (VDD), D12.3 (VDD), D13.3 (VDD), D14.3 (VDD), D15.3 (VDD), D16.3 (VDD), D17.3 (VDD), D18.3 (VDD), D19.3 (VDD), D20.3 (VDD), D21.3 (VDD), D22.3 (VDD), D23.3 (VDD), D24.3 (VDD), D9.3 (VDD), Q1.3 (D)
- new net D_N: R3.1, U1.19 (PA10/PA11/USB_D-)
- new net D_P: R4.1, U1.20 (PA12/USB_D+)
- new net MCU_PA3: R14.2, U1.9 (PA3), U3.2
- no-connect marks 18 -> 13
Other:
- note added: ""big" power reservoir for 4 SK6812 to stabilize"
- note added: "AO3401 is a power on/off switch. MMBT3904 allows MCU to switch on power for SK6812 by driving PB0 high or low (helps brownout protection at power on)"
- note added: "Convert 4.65V to 3.3V for MCU"
- note added: "Decoupling capacitors for MCU"
- note added: "Measure CC voltage"
- note added: "Status Indicator LED (active high)"
- note added: "USB LEDs Module 16x SK6812 RGBW"
- note added: "VBUS sensing, measure voltage (could be left unpopulated)"
- note added: "WS2812 decides "1" at 0.7 of own supply voltage. Supply voltage at 5V, *0.7 = 3.5V threshold. MCU sends a "1" at 3.3V -> below threshold, LED would never see a "1". This chip "converts" data signal from MCU to a clear +5V for "1" so data signal is unambiguous towards SK6812."
- note added: "bypass capacitor for each SK6812 to stabilize power"
- note added: "optional to add Ferrite Bead (600R@100Mhz - LCSC C275451) between 3.3V and VDDA to improve ADC for USB sensing"
- note added: "protect BL9110 reverse charge"
- note removed: ""big" power reservoir for 4 WS2812b to stabilize"
- note removed: "Bulk capacitors for XC6206P"
- note removed: "Convert 4.1V to 3.3V"
- note removed: "Decoupling capacitor for MCU"
- note removed: "bypass capacitor for each WS2812B to stabilize power"
- note removed: "decoupling capacitor for 4 WS2812b to stabilize"
- note removed: "protect XC6206P reverse charge"
- title: USB-C LED Module -> USB-C LEDs Module
- moved on the sheet: C1, C10, C11, C12, C13, C14, C15, C16, C17, C18, C2, C3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
